File: BM1366.kicad_pcb (KiCad board)
At the start: 2 copper layers, 1 part, among them U1 TPS4030x

Commit message: did some stuffs
Parts:
- added C1: 47uF, Capacitor_SMD:C_1210_3225Metric, F.Cu at (206.1, 125.2)
- added C2: 47uF, Capacitor_SMD:C_1210_3225Metric, F.Cu at (206.1, 129.4)
- added C3: 47uF, Capacitor_SMD:C_1210_3225Metric, F.Cu at (206.1, 133.7)
- added C4: 1uF, Capacitor_SMD:C_0805_2012Metric, F.Cu at (211.1, 129.6)
- added C5: 3.3nF, Capacitor_SMD:C_0402_1005Metric, F.Cu at (210.3, 132.1)
- added C6: 1.5nF, Capacitor_SMD:C_0805_2012Metric, F.Cu at (218.0, 129.5)
- added C7: 180pF, Capacitor_SMD:C_0805_2012Metric, F.Cu at (221.0, 129.5)
- added C8: 0.1uF, Capacitor_SMD:C_0402_1005Metric, F.Cu at (215.6, 113.9)
- added C9: 10uF, Capacitor_SMD:C_0805_2012Metric, F.Cu at (212.4, 119.4)
- added L1: 150nH, Library:FP1005R1-R15-R, F.Cu at (232.8, 116.8)
- added Q1: CSD17311Q5, Library:CSD17576Q5B, F.Cu at (229.7, 131.1)
- added Q2: CSD17311Q5, Library:CSD17576Q5B, F.Cu at (230.6, 123.0)
- added Q3: 2N7002K, Package_TO_SOT_SMD:SOT-323_SC-70, F.Cu at (204.7, 116.8)
- added R1: 3.83k, Resistor_SMD:R_0402_1005Metric, F.Cu at (215.5, 128.8)
- added R2: 4.12k, Resistor_SMD:R_0402_1005Metric, F.Cu at (205.2, 109.2)
- moved U1 201.7 mm to (217.0, 110.8)
Connections:
- U1 pad 1: unconnected-(U1-VDD-Pad1) -> Net-(J1-Pin_1)
- U1 pad 10: unconnected-(U1-BP-Pad10) -> Net-(U1-BP)
- U1 pad 11: unconnected-(U1-GND-Pad11) -> Earth
- U1 pad 2: unconnected-(U1-EN/SS-Pad2) -> Net-(Q3-D)
- U1 pad 3: unconnected-(U1-PGOOD-Pad3) -> /PGOOD
- U1 pad 4: unconnected-(U1-COMP-Pad4) -> Net-(U1-COMP)
- U1 pad 5: unconnected-(U1-FB-Pad5) -> Net-(U1-FB)
- U1 pad 6: unconnected-(U1-BOOT-Pad6) -> Net-(U1-BOOT)
- U1 pad 7: unconnected-(U1-HDRV-Pad7) -> Net-(Q1-G)
- U1 pad 8: unconnected-(U1-SW-Pad8) -> Net-(Q1-S)
- U1 pad 9: unconnected-(U1-LDRV-Pad9) -> Net-(Q2-G)
